File: electronics/crabsy_electronics.kicad_sch (KiCad schematic)
At the start: 89 parts, among them J1 Conn_01x03_Pin, J10 Conn_01x03_Pin, J11 Conn_01x03_Pin, J12 Conn_01x03_Pin, J13 Conn_01x03_Pin, J14 Conn_01x03_Pin, J15 Conn_01x03_Pin, J16 Conn_01x03_Pin, J17 Conn_01x03_Socket, J18 Conn_01x03_Socket, J19 Conn_01x03_Socket, J2 Conn_01x03_Pin, J20 Conn_01x03_Socket, J21 Conn_01x03_Socket, J22 Conn_01x03_Socket, J23 Conn_01x03_Socket, J24 Conn_01x03_Socket, J25 Conn_01x03_Socket, J26 Conn_01x03_Pin, J27 Conn_01x03_Pin, J28 Conn_01x03_Pin, J29 Conn_01x03_Pin, J3 Conn_01x03_Pin, J30 Conn_01x03_Pin, J31 Conn_01x03_Pin, J32 Conn_01x03_Pin, J35 Conn_01x03_Pin, J36 Conn_01x03_Pin, J37 Conn_01x03_Pin, J38 Conn_01x03_Pin, J39 Conn_01x03_Pin, J4 Conn_01x03_Pin, J40 Conn_01x03_Pin, J41 Conn_01x03_Pin, J42 Conn_01x03_Pin, J43 Conn_01x03_Pin, J44 Conn_01x03_Socket, J45 Conn_01x03_Socket, J46 Conn_01x03_Socket, J47 Conn_01x03_Socket, J48 Conn_01x03_Socket, J49 Conn_01x03_Socket, J5 Conn_01x03_Pin, J50 Conn_01x03_Socket, J51 Conn_01x03_Socket, J52 Conn_01x03_Socket, J54 USB_A, J6 Conn_01x03_Pin, J7 Conn_01x03_Pin, J8 Conn_01x03_Pin, J9 Conn_01x03_Pin, M1 Motor_Servo, M10 Motor_Servo, M11 Motor_Servo, M12 Motor_Servo, M13 Motor_Servo, M14 Motor_Servo, M15 Motor_Servo, M16 Motor_Servo, M17 Motor_Servo, M18 Motor_Servo, M2 Motor_Servo, M3 Motor_Servo, M4 Motor_Servo, M5 Motor_Servo, M6 Motor_Servo, M7 Motor_Servo, M8 Motor_Servo, M9 Motor_Servo, U2 PCA9685PW, U4 ESP32-WROOM-32, U5 PCA9685PW, U6 MPU-6000, U7 OPA340NA

Commit message: updating schematics
Parts:
- removed E-A1.U2.U2, E-A1.U2.U3: ATA00AA18S-L, Converter_DCDC:Converter_DCDC_Artesyn_ATA_SMD, symbol Converter_DCDC:ATA00AA18S-L
Connections:
- net +5V: now also E-A1.U2.U1.9 (+VOUT), U2.28 (VDD), U5.28 (VDD)
- net +6V renamed +VDC
- net +VDC: no longer E-A1.U2.U1.9 (+VOUT), U2.28 (VDD), U5.28 (VDD)
- no-connect marks 23 -> 19
Other:
- note removed: "POWER SUPPLY The power supply has 3 DC-DC Converters, each with a maximum output of 3 Amp. Each servo driver board gets it's own converter (6V), aswell as the logic (5V)"
- moved on the sheet: BZ1, C1, C2, D1, MK1, R1, R2, R3, R4, U6, U7
